Commit message: Remove depth camera configuration from xArm7 URDF

File: xarm_description/urdf/xarm7/xarm7.urdf.xacro (robot description, xacro)
@@ -281,65 +281,4 @@
       <child link="${prefix}link_eef" />
     </joint> -->
-    <!-- Depth Camera: Intel RealSense D435 with Stand -->
-  <link name="depth_camera_link">
-    <visual>
-      <origin xyz="0 0 0" rpy="0 0 0"/>
-      <geometry>
-        <mesh filename="package://xarm_description/meshes/camera/realsense/visual/d435_with_cam_stand.stl" scale="0.001 0.001 0.001"/>
-      </geometry>
-    </visual>
-    <collision>
-      <origin xyz="0 0 0" rpy="0 0 0"/>
-      <geometry>
-        <mesh filename="package://xarm_description/meshes/camera/realsense/collision/d435_with_cam_stand.stl" scale="0.001 0.001 0.001"/>
-      </geometry>
-    </collision>
-    <inertial>
-      <mass value="0.1"/>
-      <origin xyz="0 0 0" rpy="0 0 0"/>
-      <inertia ixx="1e-5" ixy="0" ixz="0" iyy="1e-5" iyz="0" izz="1e-5"/>
-    </inertial>
-  </link>
-  <joint name="depth_camera_joint" type="fixed">
-    <parent link="${prefix}link_base"/>
-    <child link="depth_camera_link"/>
-    <origin xyz="0 0 0.12" rpy="0 0 0"/>
-  </joint>
-  <!-- Gazebo Plugin for Depth Camera -->
-  <gazebo reference="depth_camera_link">
-    <sensor name="depth_camera_sensor" type="depth">
-      <pose>0 0 0 0 0 0</pose>
-      <visualize>true</visualize>
-      <update_rate>30.0</update_rate>
-      <camera>
-        <horizontal_fov>1.39626</horizontal_fov> <!-- ~80 deg -->
-        <image>
-          <width>640</width>
-          <height>480</height>
-          <format>R8G8B8</format>
-        </image>
-        <clip>
-          <near>0.1</near>
-          <far>5.0</far>
-        </clip>
-        <noise>
-          <type>gaussian</type>
-          <mean>0.0</mean>
-          <stddev>0.007</stddev>
-        </noise>
-      </camera>
-      <!-- Plugin -->
-      <plugin name="gazebo_ros_depth_camera" filename="libgazebo_ros_depth_camera.so">
-        <ros>
-          <namespace>/depth_camera</namespace>
-        </ros>
-        <camera_name>depth_camera</camera_name>
-        <image_topic_name>rgb/image_raw</image_topic_name>
-        <depth_image_topic_name>depth/image_raw</depth_image_topic_name>
-        <camera_info_topic_name>camera_info</camera_info_topic_name>
-        <frame_name>depth_camera_link</frame_name>
-      </plugin>
-    </sensor>
-  </gazebo>
   </xacro:macro>
 </robot>
