Commit message: Add new models and configurations for box and bookshelf in Gazebo

File: xarm_moveit_config/srdf/_xarm7_macro.srdf.xacro (robot description, xacro)
@@ -57,4 +57,13 @@
       <joint name="${prefix}joint6" value="-1.5708" />
       <joint name="${prefix}joint7" value="0" />
+    </group_state>
+      <group_state name="look" group="${prefix}xarm7">
+      <joint name="${prefix}joint1" value="-9.634109314315964e-05" />
+      <joint name="${prefix}joint2" value="-0.071963249884918312" />
+      <joint name="${prefix}joint3" value="-0.00017165762239823579" />
+      <joint name="${prefix}joint4" value="1.6127273478062465" />
+      <joint name="${prefix}joint5" value="-6.3550559483260827e-05" />
+      <joint name="${prefix}joint6" value="1.6576269636020662" />
+      <joint name="${prefix}joint7" value="-0.00015535496839191865" />
     </group_state>
     <!-- gripper -->

Commit message: Add xarm7_aruco_pick package with ArUco detection functionality and configuration

File: xarm_moveit_config/srdf/_xarm7_macro.srdf.xacro (robot description, xacro)
@@ -58,5 +58,5 @@
       <joint name="${prefix}joint7" value="0" />
     </group_state>
-      <group_state name="look" group="${prefix}xarm7">
+    <group_state name="look" group="${prefix}xarm7">
       <joint name="${prefix}joint1" value="-9.634109314315964e-05" />
       <joint name="${prefix}joint2" value="-0.071963249884918312" />
@@ -66,4 +66,94 @@
       <joint name="${prefix}joint6" value="1.6576269636020662" />
       <joint name="${prefix}joint7" value="-0.00015535496839191865" />
+    </group_state>
+    <group_state name="hold_1" group="${prefix}xarm7">
+      <joint name="${prefix}joint1" value="4.0654922539827727e-05" />
+      <joint name="${prefix}joint2" value="-0.37657474678886493" />
+      <joint name="${prefix}joint3" value="5.7346847492034669e-05" />
+      <joint name="${prefix}joint4" value="0.93885744778211055" />
+      <joint name="${prefix}joint5" value="4.8938829047926702e-05" />
+      <joint name="${prefix}joint6" value="1.315498315216959" />
+      <joint name="${prefix}joint7" value="-8.5591281735681931e-05" />
+    </group_state>
+    <group_state name="hold_2" group="${prefix}xarm7">
+      <joint name="${prefix}joint1" value="-0.2032961155294124" />
+      <joint name="${prefix}joint2" value="-0.54983707354786282" />
+      <joint name="${prefix}joint3" value="1.0015727395430529" />
+      <joint name="${prefix}joint4" value="0.27488056214633172" />
+      <joint name="${prefix}joint5" value="0.92198869447854293" />
+      <joint name="${prefix}joint6" value="-0.80650243703676505" />
+      <joint name="${prefix}joint7" value="-0.13503031427615464" />
+    </group_state>
+    <group_state name="look" group="${prefix}xarm7">
+      <joint name="${prefix}joint1" value="-9.634109314315964e-05" />
+      <joint name="${prefix}joint2" value="-0.071963249884918312" />
+      <joint name="${prefix}joint3" value="-0.00017165762239823579" />
+      <joint name="${prefix}joint4" value="1.6127273478062465" />
+      <joint name="${prefix}joint5" value="-6.3550559483260827e-05" />
+      <joint name="${prefix}joint6" value="1.6576269636020662" />
+      <joint name="${prefix}joint7" value="-0.00015535496839191865" />
+    </group_state>
+    <group_state name="pick" group="${prefix}xarm7">
+      <joint name="${prefix}joint1" value="-0.286933154016493" />
+      <joint name="${prefix}joint2" value="0.67706222921724657" />
+      <joint name="${prefix}joint3" value="0.928213309820074" />
+      <joint name="${prefix}joint4" value="1.2962469247696964" />
+      <joint name="${prefix}joint5" value="0.55061019503566211" />
+      <joint name="${prefix}joint6" value="-1.0351266277916258" />
+      <joint name="${prefix}joint7" value="-0.87474288709510417" />
+    </group_state>
+    <group_state name="up_1" group="${prefix}xarm7">
+      <joint name="${prefix}joint1" value="0.081479226265743998" />
+      <joint name="${prefix}joint2" value="0.24329056521030279" />
+      <joint name="${prefix}joint3" value="0.12793005353051523" />
+      <joint name="${prefix}joint4" value="1.8787746088121366" />
+      <joint name="${prefix}joint5" value="-1.1115896149302049" />
+      <joint name="${prefix}joint6" value="0.23105475637973338" />
+      <joint name="${prefix}joint7" value="1.0784426530478408" />
+    </group_state>
+    <group_state name="drop_pre" group="${prefix}xarm7">
+      <joint name="${prefix}joint1" value="-0.16724176176672478" />
+      <joint name="${prefix}joint2" value="-0.29796048652525164" />
+      <joint name="${prefix}joint3" value="-0.3324480460038135" />
+      <joint name="${prefix}joint4" value="1.7778865017393706" />
+      <joint name="${prefix}joint5" value="0.16952947148145636" />
+      <joint name="${prefix}joint6" value="1.558199022746841" />
+      <joint name="${prefix}joint7" value="-0.46908596267092117" />
+    </group_state>
+    <group_state name="drop_pre2" group="${prefix}xarm7">
+      <joint name="${prefix}joint1" value="0.031986571227971661" />
+      <joint name="${prefix}joint2" value="-0.42298497966572746" />
+      <joint name="${prefix}joint3" value="-0.99625700117549165" />
+      <joint name="${prefix}joint4" value="1.2969742695315425" />
+      <joint name="${prefix}joint5" value="-0.49931511306467069" />
+      <joint name="${prefix}joint6" value="1.6063673293155531" />
+      <joint name="${prefix}joint7" value="-0.89890753554889247" />
+    </group_state>
+    <group_state name="dropped" group="${prefix}xarm7">
+      <joint name="${prefix}joint1" value="0.22358179078550067" />
+      <joint name="${prefix}joint2" value="-0.87281179218304739" />
+      <joint name="${prefix}joint3" value="-1.7001430506547397" />
+      <joint name="${prefix}joint4" value="1.3801484717737704" />
+      <joint name="${prefix}joint5" value="-0.89492940575112634" />
+      <joint name="${prefix}joint6" value="1.3101577186303706" />
+      <joint name="${prefix}joint7" value="-1.2734589874875295" />
+    </group_state>
+    <group_state name="going_home" group="${prefix}xarm7">
+      <joint name="${prefix}joint1" value="-0.035197328295303754" />
+      <joint name="${prefix}joint2" value="-1.0706044648355026" />
+      <joint name="${prefix}joint3" value="0.17123786956791331" />
+      <joint name="${prefix}joint4" value="1.0033068438722204" />
+      <joint name="${prefix}joint5" value="0.10169620196486573" />
+      <joint name="${prefix}joint6" value="1.8609536265364532" />
+      <joint name="${prefix}joint7" value="0.10605600767823398" />
+    </group_state>
+    <group_state name="Home" group="${prefix}xarm7">
+      <joint name="${prefix}joint1" value="6.8717429668518903e-05" />
+      <joint name="${prefix}joint2" value="9.6140206806483164e-05" />
+      <joint name="${prefix}joint3" value="4.6904267826164414e-05" />
+      <joint name="${prefix}joint4" value="-3.6416929710014756e-05" />
+      <joint name="${prefix}joint5" value="3.7716389483577473e-05" />
+      <joint name="${prefix}joint6" value="-7.4198795978475118e-05" />
+      <joint name="${prefix}joint7" value="-5.5301690339737419e-05" />
     </group_state>
     <!-- gripper -->

Commit message: Update robot configurations and parameters for xarm7
- Changed service call parameters in ReadMe.md to use 'box_2' instead of 'box_1'.
- Updated saved joint poses in saved_joint_poses.yaml, adding new poses and removing outdated ones.
- Modified pose_saver.cpp to change the save path for joint poses.
- Added attach_detach_plugin to table.world for improved object interaction.
- Adjusted planner.rviz settings, including acceleration scaling factor and enabling Cartesian path planning.
- Updated _xarm7_macro.srdf.xacro to reflect new joint states and removed obsolete group states.

File: xarm_moveit_config/srdf/_xarm7_macro.srdf.xacro (robot description, xacro)
@@ -49,102 +49,39 @@
       <joint name="${prefix}joint7" value="0" />
     </group_state>
-    <group_state name="hold-up" group="${prefix}xarm7">
-      <joint name="${prefix}joint1" value="0" />
-      <joint name="${prefix}joint2" value="0" />
-      <joint name="${prefix}joint3" value="0" />
-      <joint name="${prefix}joint4" value="0" />
-      <joint name="${prefix}joint5" value="0" />
-      <joint name="${prefix}joint6" value="-1.5708" />
-      <joint name="${prefix}joint7" value="0" />
+    <group_state name="up" group="${prefix}xarm7">
+      <joint name="${prefix}joint1" value="3.7490367097881006e-05" />
+      <joint name="${prefix}joint2" value="-0.7557058858721275" />
+      <joint name="${prefix}joint3" value="2.2576265923390793e-06" />
+      <joint name="${prefix}joint4" value="1.177697926332379" />
+      <joint name="${prefix}joint5" value="1.1954546238257535e-05" />
+      <joint name="${prefix}joint6" value="1.9334524926102468" />
+      <joint name="${prefix}joint7" value="-1.2640088147719553e-05" />
     </group_state>
     <group_state name="look" group="${prefix}xarm7">
-      <joint name="${prefix}joint1" value="-9.634109314315964e-05" />
-      <joint name="${prefix}joint2" value="-0.071963249884918312" />
-      <joint name="${prefix}joint3" value="-0.00017165762239823579" />
-      <joint name="${prefix}joint4" value="1.6127273478062465" />
-      <joint name="${prefix}joint5" value="-6.3550559483260827e-05" />
-      <joint name="${prefix}joint6" value="1.6576269636020662" />
-      <joint name="${prefix}joint7" value="-0.00015535496839191865" />
-    </group_state>
-    <group_state name="hold_1" group="${prefix}xarm7">
-      <joint name="${prefix}joint1" value="4.0654922539827727e-05" />
-      <joint name="${prefix}joint2" value="-0.37657474678886493" />
-      <joint name="${prefix}joint3" value="5.7346847492034669e-05" />
-      <joint name="${prefix}joint4" value="0.93885744778211055" />
-      <joint name="${prefix}joint5" value="4.8938829047926702e-05" />
-      <joint name="${prefix}joint6" value="1.315498315216959" />
-      <joint name="${prefix}joint7" value="-8.5591281735681931e-05" />
-    </group_state>
-    <group_state name="hold_2" group="${prefix}xarm7">
-      <joint name="${prefix}joint1" value="-0.2032961155294124" />
-      <joint name="${prefix}joint2" value="-0.54983707354786282" />
-      <joint name="${prefix}joint3" value="1.0015727395430529" />
-      <joint name="${prefix}joint4" value="0.27488056214633172" />
-      <joint name="${prefix}joint5" value="0.92198869447854293" />
-      <joint name="${prefix}joint6" value="-0.80650243703676505" />
-      <joint name="${prefix}joint7" value="-0.13503031427615464" />
-    </group_state>
-    <group_state name="look" group="${prefix}xarm7">
-      <joint name="${prefix}joint1" value="-9.634109314315964e-05" />
-      <joint name="${prefix}joint2" value="-0.071963249884918312" />
-      <joint name="${prefix}joint3" value="-0.00017165762239823579" />
-      <joint name="${prefix}joint4" value="1.6127273478062465" />
-      <joint name="${prefix}joint5" value="-6.3550559483260827e-05" />
-      <joint name="${prefix}joint6" value="1.6576269636020662" />
-      <joint name="${prefix}joint7" value="-0.00015535496839191865" />
+      <joint name="${prefix}joint1" value="0.1388548331359134" />
+      <joint name="${prefix}joint2" value="-0.35411523916076515" />
+      <joint name="${prefix}joint3" value="-0.17444431215925871" />
+      <joint name="${prefix}joint4" value="1.4426785833000872" />
+      <joint name="${prefix}joint5" value="-0.061715033311549483" />
+      <joint name="${prefix}joint6" value="1.7915080917332666" />
+      <joint name="${prefix}joint7" value="-0.025441950871051056" />
+    </group_state>
+    <group_state name="pick_pre" group="${prefix}xarm7">
+      <joint name="${prefix}joint1" value="0.19919301702224512" />
+      <joint name="${prefix}joint2" value="0.15075026911984679" />
+      <joint name="${prefix}joint3" value="-0.18474536255557528" />
+      <joint name="${prefix}joint4" value="1.3080527313086483" />
+      <joint name="${prefix}joint5" value="0.030092487096007758" />
+      <joint name="${prefix}joint6" value="1.1600586083971107" />
+      <joint name="${prefix}joint7" value="0.017519159504584714" />
     </group_state>
     <group_state name="pick" group="${prefix}xarm7">
-      <joint name="${prefix}joint1" value="-0.286933154016493" />
-      <joint name="${prefix}joint2" value="0.67706222921724657" />
-      <joint name="${prefix}joint3" value="0.928213309820074" />
-      <joint name="${prefix}joint4" value="1.2962469247696964" />
-      <joint name="${prefix}joint5" value="0.55061019503566211" />
-      <joint name="${prefix}joint6" value="-1.0351266277916258" />
-      <joint name="${prefix}joint7" value="-0.87474288709510417" />
-    </group_state>
-    <group_state name="up_1" group="${prefix}xarm7">
-      <joint name="${prefix}joint1" value="0.081479226265743998" />
-      <joint name="${prefix}joint2" value="0.24329056521030279" />
-      <joint name="${prefix}joint3" value="0.12793005353051523" />
-      <joint name="${prefix}joint4" value="1.8787746088121366" />
-      <joint name="${prefix}joint5" value="-1.1115896149302049" />
-      <joint name="${prefix}joint6" value="0.23105475637973338" />
-      <joint name="${prefix}joint7" value="1.0784426530478408" />
-    </group_state>
-    <group_state name="drop_pre" group="${prefix}xarm7">
-      <joint name="${prefix}joint1" value="-0.16724176176672478" />
-      <joint name="${prefix}joint2" value="-0.29796048652525164" />
-      <joint name="${prefix}joint3" value="-0.3324480460038135" />
-      <joint name="${prefix}joint4" value="1.7778865017393706" />
-      <joint name="${prefix}joint5" value="0.16952947148145636" />
-      <joint name="${prefix}joint6" value="1.558199022746841" />
-      <joint name="${prefix}joint7" value="-0.46908596267092117" />
-    </group_state>
-    <group_state name="drop_pre2" group="${prefix}xarm7">
-      <joint name="${prefix}joint1" value="0.031986571227971661" />
-      <joint name="${prefix}joint2" value="-0.42298497966572746" />
-      <joint name="${prefix}joint3" value="-0.99625700117549165" />
-      <joint name="${prefix}joint4" value="1.2969742695315425" />
-      <joint name="${prefix}joint5" value="-0.49931511306467069" />
-      <joint name="${prefix}joint6" value="1.6063673293155531" />
-      <joint name="${prefix}joint7" value="-0.89890753554889247" />
-    </group_state>
-    <group_state name="dropped" group="${prefix}xarm7">
-      <joint name="${prefix}joint1" value="0.22358179078550067" />
-      <joint name="${prefix}joint2" value="-0.87281179218304739" />
-      <joint name="${prefix}joint3" value="-1.7001430506547397" />
-      <joint name="${prefix}joint4" value="1.3801484717737704" />
-      <joint name="${prefix}joint5" value="-0.89492940575112634" />
-      <joint name="${prefix}joint6" value="1.3101577186303706" />
-      <joint name="${prefix}joint7" value="-1.2734589874875295" />
-    </group_state>
-    <group_state name="going_home" group="${prefix}xarm7">
-      <joint name="${prefix}joint1" value="-0.035197328295303754" />
-      <joint name="${prefix}joint2" value="-1.0706044648355026" />
-      <joint name="${prefix}joint3" value="0.17123786956791331" />
-      <joint name="${prefix}joint4" value="1.0033068438722204" />
-      <joint name="${prefix}joint5" value="0.10169620196486573" />
-      <joint name="${prefix}joint6" value="1.8609536265364532" />
-      <joint name="${prefix}joint7" value="0.10605600767823398" />
+      <joint name="${prefix}joint1" value="0.19350702274674969" />
+      <joint name="${prefix}joint2" value="0.26299530657961601" />
+      <joint name="${prefix}joint3" value="-0.17779503075125014" />
+      <joint name="${prefix}joint4" value="1.1456634297516803" />
+      <joint name="${prefix}joint5" value="0.059317746340783017" />
+      <joint name="${prefix}joint6" value="0.88755047346460092" />
+      <joint name="${prefix}joint7" value="-0.0027309607560068727" />
     </group_state>
     <group_state name="Home" group="${prefix}xarm7">
@@ -156,4 +93,40 @@
       <joint name="${prefix}joint6" value="-7.4198795978475118e-05" />
       <joint name="${prefix}joint7" value="-5.5301690339737419e-05" />
+    </group_state>
+    <group_state name="drop_post" group="${prefix}xarm7">
+      <joint name="${prefix}joint1" value="0.034168209390873727" />
+      <joint name="${prefix}joint2" value="0.27173424338337426" />
+      <joint name="${prefix}joint3" value="-0.010816053136127657" />
+      <joint name="${prefix}joint4" value="2.1031429110457474" />
+      <joint name="${prefix}joint5" value="0.003005323964641704" />
+      <joint name="${prefix}joint6" value="1.8315049015911793" />
+      <joint name="${prefix}joint7" value="0.03756073234481061" />
+    </group_state>
+    <group_state name="drop_pre" group="${prefix}xarm7">
+      <joint name="${prefix}joint1" value="-0.72484240195298888" />
+      <joint name="${prefix}joint2" value="-0.35561185672245088" />
+      <joint name="${prefix}joint3" value="-0.9727001693241224" />
+      <joint name="${prefix}joint4" value="1.5924088368430729" />
+      <joint name="${prefix}joint5" value="-0.29919658361787693" />
+      <joint name="${prefix}joint6" value="1.7887907297988779" />
+      <joint name="${prefix}joint7" value="-0.2476618179822907" />
+    </group_state>
+    <group_state name="drop" group="${prefix}xarm7">
+      <joint name="${prefix}joint1" value="-0.70230505955947553" />
+      <joint name="${prefix}joint2" value="-0.3860187216760238" />
+      <joint name="${prefix}joint3" value="-1.2475438702204169" />
+      <joint name="${prefix}joint4" value="0.77749837556607293" />
+      <joint name="${prefix}joint5" value="-0.45216461018011067" />
+      <joint name="${prefix}joint6" value="0.95658329312072876" />
+      <joint name="${prefix}joint7" value="-0.16708702185973934" />
+    </group_state>
+    <group_state name="home_pre" group="${prefix}xarm7">
+      <joint name="${prefix}joint1" value="-0.30938962196237885" />
+      <joint name="${prefix}joint2" value="-0.51193327711608205" />
+      <joint name="${prefix}joint3" value="0.23820317565758842" />
+      <joint name="${prefix}joint4" value="1.1455434196811805" />
+      <joint name="${prefix}joint5" value="0.11617213185493114" />
+      <joint name="${prefix}joint6" value="1.6448678872791591" />
+      <joint name="${prefix}joint7" value="-0.092139458728333956" />
     </group_state>
     <!-- gripper -->
